File: Earphones_amp.kicad_sch (KiCad schematic)
At the start: 75 parts, among them J1 AudioJack3, J2 AudioJack3, Q1 2SC1815, Q10 PNP, Q2 2SA1015, Q3 PNP, Q4 NPN, Q5 PNP, Q6 NPN, Q7 NPN, Q8 PNP, Q9 NPN, U1 Opamp_Dual, U2 TL072, U3 TL074, U4 OPA1655DR, U5 TL074

Commit message: 部品置いた
Connections:
- net sigIN_L: now also U2.3 (+); no longer U2.5 (+)
- net sigIN_R: now also U2.5 (+); no longer U2.3 (+)
- net at C13.2, R17.1: now also U3.12 (+); no longer U3.10 (+)
- net at R5.2, RV1.3, RV2.3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: now also U3.10 (+); no longer U3.12 (+)
- net at R19.1, RV1.1, RV2.1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: now also U3.9 (-); no longer U3.13 (-)
- net at R19.2, RV4.1: now also U3.8; no longer U3.14
- net outL renamed out_L
- net out_L: now also R23.2, R35.2
- net outR renamed out_R
- net out_R: no longer R23.2, R35.2
- new net: R15.2, U3.13 (-), U3.14
Other:
- moved on the sheet: J1, U3C, U3D
Changed lines of the file:
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@@
 	)
 	(junction
-		(at 140.97 77.47)
-		(diameter 0)
-		(color 0 0 0 0)
-	)
-	(junction
 		(at 209.55 130.81)
 		(diameter 0)
@@
 	)
 	(junction
-		(at 135.89 77.47)
-		(diameter 0)
-		(color 0 0 0 0)
-	)
-	(junction
 		(at 146.05 53.34)
 		(diameter 0)
@@
 	)
 	(junction
+		(at 135.89 77.47)
+		(diameter 0)
+		(color 0 0 0 0)
+	)
+	(junction
 		(at -17.78 97.79)
 		(diameter 0)
@@
 	)
 	(junction
-		(at 161.29 57.15)
-		(diameter 0)
-		(color 0 0 0 0)
-	)
-	(junction
 		(at -17.78 107.95)
 		(diameter 0)
@@
 	)
 	(junction
+		(at 161.29 57.15)
+		(diameter 0)
+		(color 0 0 0 0)
+	)
+	(junction
 		(at 80.01 77.47)
 		(diameter 0)
@@
 	)
 	(junction
+		(at 140.97 77.47)
+		(diameter 0)
+		(color 0 0 0 0)
+	)
+	(junction
 		(at 173.99 91.44)
 		(diameter 0)
@@
 		)
 	)
+	(label "out_R"
+		(at 261.62 100.33 180)
+		(effects
+			(font
+				(size 1.27 1.27)
+			)
+			(justify right bottom)
+		)
+	)
 	(label "V_{+}"
 		(at -6.35 87.63 0)
@@
 		)
 	)
-	(label "outR"
+	(label "out_R"
 		(at 242.57 119.38 0)
 		(effects
@@
 	)
 	(label "sigIN_L"
-		(at 38.1 91.44 0)
+		(at -44.45 144.78 0)
 		(effects
 			(font
@@
 	)
 	(label "sigIN_R"
-		(at 38.1 93.98 0)
+		(at -44.45 147.32 0)
 		(effects
 			(font
@@
 		)
 	)
-	(label "outR"
-		(at 261.62 100.33 180)
-		(effects
-			(font
-				(size 1.27 1.27)
-			)
-			(justify right bottom)
-		)
-	)
 	(label "V_{+}"
 		(at 76.2 180.34 0)
@@
 		)
 	)
-	(label "outL"
-		(at 261.62 97.79 180)
-		(effects
-			(font
-				(size 1.27 1.27)
-			)
-			(justify right bottom)
-		)
-	)
 	(label "V_{+}"
 		(at 41.91 180.34 0)
@@
 		)
 	)
-	(label "sigIN_R"
+	(label "sigIN_L"
 		(at 49.53 58.42 180)
 		(effects
@@
 		)
 	)
-	(label "outR"
+	(label "out_L"
 		(at 242.57 63.5 0)
 		(effects
@@
 		)
 	)
+	(label "out_L"
+		(at 261.62 97.79 180)
+		(effects
+			(font
+				(size 1.27 1.27)
+			)
+			(justify right bottom)
+		)
+	)
 	(label "V_{-}"
 		(at 76.2 195.58 0)
@@
 		)
 	)
-	(label "sigIN_L"
+	(label "sigIN_R"
 		(at 49.53 114.3 180)
 		(effects
@@
 	(symbol
 		(lib_id "Device:Opamp_Quad")
-		(at 138.43 85.09 270)
+		(at 153.67 57.15 0)
+		(mirror x)
 		(unit 3)
 		(body_style 1)
@@
 		(dnp no)
 		(property "Reference" "U3"
-			(at 132.08 83.82 90)
+			(at 153.67 65.532 0)
 			(show_name no)
 			(do_not_autoplace no)
@@
 					(size 1.27 1.27)
 				)
-				(justify right)
 			)
 		)
 		(property "Value" "TL074"
-			(at 132.08 86.36 90)
+			(at 153.67 62.992 0)
 			(show_name no)
 			(do_not_autoplace no)
@@
 					(size 1.27 1.27)
 				)
-				(justify right)
 			)
 		)
 		(property "Footprint" "Package_DIP:DIP-14_W7.62mm_Socket"
-			(at 138.43 85.09 0)
+			(at 153.67 57.15 0)
 			(hide yes)
 			(show_name no)
@@
 		)
 		(property "Datasheet" ""
-			(at 138.43 85.09 0)
+			(at 153.67 57.15 0)
 			(hide yes)
 			(show_name no)
@@
 		)
 		(property "Description" "Quad operational amplifier"
-			(at 138.43 85.09 0)
+			(at 153.67 57.15 0)
 			(hide yes)
 			(show_name no)
@@
 		)
 		(property "Sim.Library" "${KICAD9_SYMBOL_DIR}/Simulation_SPICE.sp"
-			(at 138.43 85.09 0)
+			(at 153.67 57.15 0)
 			(hide yes)
 			(show_name no)
@@
 		)
 		(property "Sim.Name" "kicad_builtin_opamp_quad"
-			(at 138.43 85.09 0)
+			(at 153.67 57.15 0)
 			(hide yes)
 			(show_name no)
@@
 		)
 		(property "Sim.Device" "SUBCKT"
-			(at 138.43 85.09 0)
+			(at 153.67 57.15 0)
 			(hide yes)
 			(show_name no)
@@
 		)
 		(property "Sim.Pins" "1=out1 2=in1- 3=in1+ 4=vcc 5=in2+ 6=in2- 7=out2 8=out3 9=in3- 10=in3+ 11=vee 12=in4+ 13=in4- 14=out4"
-			(at 138.43 85.09 0)
+			(at 153.67 57.15 0)
 			(hide yes)
 			(show_name no)
@@
 	(symbol
 		(lib_id "Device:Opamp_Quad")
-		(at 153.67 57.15 0)
-		(mirror x)
+		(at 138.43 85.09 270)
 		(unit 4)
 		(body_style 1)
@@
 		(dnp no)
 		(property "Reference" "U3"
-			(at 153.67 66.04 0)
+			(at 132.08 83.82 90)
 			(show_name no)
 			(do_not_autoplace no)
@@
 					(size 1.27 1.27)
 				)
+				(justify right)
 			)
 		)
 		(property "Value" "TL074"
-			(at 153.67 63.5 0)
+			(at 132.08 86.36 90)
 			(show_name no)
 			(do_not_autoplace no)
@@
 					(size 1.27 1.27)
 				)
+				(justify right)
 			)
 		)
 		(property "Footprint" "Package_DIP:DIP-14_W7.62mm_Socket"
-			(at 153.67 57.15 0)
+			(at 138.43 85.09 0)
 			(hide yes)
 			(show_name no)
@@
 		)
 		(property "Datasheet" ""
-			(at 153.67 57.15 0)
+			(at 138.43 85.09 0)
 			(hide yes)
 			(show_name no)
@@
 		)
 		(property "Description" "Quad operational amplifier"
-			(at 153.67 57.15 0)
+			(at 138.43 85.09 0)
 			(hide yes)
 			(show_name no)
@@
 		)
 		(property "Sim.Library" "${KICAD9_SYMBOL_DIR}/Simulation_SPICE.sp"
-			(at 153.67 57.15 0)
+			(at 138.43 85.09 0)
 			(hide yes)
 			(show_name no)
@@
 		)
 		(property "Sim.Name" "kicad_builtin_opamp_quad"
-			(at 153.67 57.15 0)
+			(at 138.43 85.09 0)
 			(hide yes)
 			(show_name no)
@@
 		)
 		(property "Sim.Device" "SUBCKT"
-			(at 153.67 57.15 0)
+			(at 138.43 85.09 0)
 			(hide yes)
 			(show_name no)
@@
 		)
 		(property "Sim.Pins" "1=out1 2=in1- 3=in1+ 4=vcc 5=in2+ 6=in2- 7=out2 8=out3 9=in3- 10=in3+ 11=vee 12=in4+ 13=in4- 14=out4"
-			(at 153.67 57.15 0)
+			(at 138.43 85.09 0)
 			(hide yes)
 			(show_name no)
@@
 	(symbol
 		(lib_id "Connector_Audio:AudioJack3")
-		(at 33.02 93.98 0)
+		(at -49.53 147.32 0)
 		(mirror x)
 		(unit 1)
@@
 		(fields_autoplaced yes)
 		(property "Reference" "J1"
-			(at 25.4 92.0749 0)
+			(at -57.15 145.4149 0)
 			(show_name no)
 			(do_not_autoplace no)
@@
 		)
 		(property "Value" "AudioJack3"
-			(at 25.4 94.6149 0)
+			(at -57.15 147.9549 0)
 			(show_name no)
 			(do_not_autoplace no)
@@
 		)
 		(property "Footprint" "MyLibrary:MJ352W"
-			(at 33.02 93.98 0)
+			(at -49.53 147.32 0)
 			(hide yes)
 			(show_name no)
@@
 		)
 		(property "Datasheet" ""
-			(at 33.02 93.98 0)
+			(at -49.53 147.32 0)
 			(hide yes)
 			(show_name no)
@@
 		)
 		(property "Description" "Audio Jack, 3 Poles (Stereo / TRS)"
-			(at 33.02 93.98 0)
+			(at -49.53 147.32 0)
 			(hide yes)
 			(show_name no)
@@
 	(symbol
 		(lib_id "power:GNDREF")
-		(at 38.1 96.52 0)
+		(at -44.45 149.86 0)
 		(mirror y)
 		(unit 1)
@@
 		(dnp no)
 		(property "Reference" "#PWR03"
-			(at 38.1 102.87 0)
+			(at -44.45 156.21 0)
 			(hide yes)
 			(show_name no)
@@
 		)
 		(property "Value" "GNDREF"
-			(at 38.1 100.33 0)
+			(at -44.45 153.67 0)
 			(show_name no)
 			(do_not_autoplace no)
@@
 		)
 		(property "Footprint" ""
-			(at 38.1 96.52 0)
+			(at -44.45 149.86 0)
 			(hide yes)
 			(show_name no)
@@
 		)
 		(property "Datasheet" ""
-			(at 38.1 96.52 0)
+			(at -44.45 149.86 0)
 			(hide yes)
 			(show_name no)
@@
 		)
 		(property "Description" "Power symbol creates a global label with name \"GNDREF\" , reference supply ground"
-			(at 38.1 96.52 0)
+			(at -44.45 149.86 0)
 			(hide yes)
 			(show_name no)

Commit message: gbr出力
Parts:
- added C15, C16, C17, C18, C19: 0.1u, Capacitor_THT:C_Disc_D5.1mm_W3.2mm_P5.00mm, symbol Device:C
- added SW1: SW_SPDT, samacsys:SS12D00G3, symbol Switch:SW_SPDT
- D1: footprint LED_THT:LED_D5.0mm -> LED_THT:LED_D3.0mm_Horizontal_O1.27mm_Z2.0mm
Connections:
- net V_{+}: now also C15.1, C16.1, C17.1, C18.1, C19.1, SW1.1 (A); no longer BT1.1 (+), U5.11 (V-)
- net V_{-}: now also U5.11 (V-), C15.2, C16.2, C17.2, C18.2, C19.2
- net at R19.2, U3.8: now also RV4.4; no longer RV4.1
- net at R20.2, U5.14: now also RV4.1; no longer RV4.4
- net at RV4.5: now also U4.3 (+); no longer U4.5 (+)
- net at RV4.2: now also U4.5 (+); no longer U4.3 (+)
- new net: BT1.1 (+), SW1.2 (B)
- no-connect marks 0 -> 1
Other:
- moved on the sheet: BT1, RV4A, RV4B, U2C, U3E, U4C, U5E
