File: Earphones_amp.kicad_sch (KiCad schematic)
At the start: 81 parts, among them J1 AudioJack3, J2 AudioJack3, Q1 2SC1815, Q10 PNP, Q2 2SA1015, Q3 PNP, Q4 NPN, Q5 PNP, Q6 NPN, Q7 NPN, Q8 PNP, Q9 NPN, SW1 SW_SPDT, U1 Opamp_Dual, U2 TL072, U3 TL074, U4 OPA1655DR, U5 TL074

Commit message: 回路図修正，v2.0に更新
Parts:
- added C20, C21: 0.1u, Capacitor_THT:C_Disc_D4.7mm_W2.5mm_P5.00mm, symbol Device:C
- added H1, H2, H3: MountingHole_Pad, MountingHole:MountingHole_3.2mm_M3_Pad_Via, symbol Mechanical:MountingHole_Pad
- added R37, R38: 100k, Resistor_THT:R_Axial_DIN0204_L3.6mm_D1.6mm_P5.08mm_Horizontal, symbol Device:R_Small
- D1: footprint LED_THT:LED_D3.0mm_Horizontal_O1.27mm_Z2.0mm -> LED_THT:LED_D5.0mm_Horizontal_O1.27mm_Z3.0mm
- R1: value 2k -> 10k
Connections:
- net GNDREF: now also C20.2, C21.1, H1.1, H2.1, H3.1, R37.2, R38.2
- net V_{+}: now also C20.1
- net V_{-}: now also Q10.2 (C), Q3.2 (C), Q5.2 (C), Q8.2 (C), C21.2; no longer Q10.1 (E), Q3.1 (E), Q5.1 (E), Q8.1 (E)
- net sigIN_L: now also R37.1
- net sigIN_R: now also R38.1
- net at R32.2: now also Q8.1 (E); no longer Q8.2 (C)
- net at R34.2: now also Q10.1 (E); no longer Q10.2 (C)
- net at Q9.3 (B), R29.2: now also Q5.1 (E); no longer Q5.2 (C)
- net at Q7.3 (B), R27.2: now also Q3.1 (E); no longer Q3.2 (C)
Other:
- note removed: "30mA"
- note removed: "FET入力 2回路入買ってRLで共通"
- note removed: "U3~6 4回路入 低ノイズ RLで2つ"
- note removed: "いいヤツ すでに家にある"
- note removed: "分離抵抗"
- moved on the sheet: BT1, C1, C10, C11, C12, C13, C14, C15, C16, C17, C18, C19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

Commit message: 回路図更新
Parts:
- U1: value Opamp_Dual -> LM358N
Changed lines of the file:
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@@
 			)
 		)
-		(property "Value" "Opamp_Dual"
-			(at 60.96 41.148 0)
+		(property "Value" "LM358N"
+			(at 58.928 41.148 0)
 			(show_name no)
 			(do_not_autoplace no)
@@
 			)
 		)
-		(property "Value" "Opamp_Dual"
+		(property "Value" "LM358N"
 			(at 54.864 29.972 0)
 			(show_name no)
@@
 			)
 		)
-		(property "Value" "Opamp_Dual"
+		(property "Value" "LM358N"
 			(at 29.21 179.07 0)
 			(show_name no)
