File: Earphones_amp.kicad_pcb (KiCad board)
At the start: 2 copper layers, 75 parts, among them J1 AudioJack3, J2 AudioJack3, Q1 2SC1815, Q10 PNP, Q2 2SA1015, Q3 PNP, Q4 NPN, Q5 PNP, Q6 NPN, Q7 NPN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

Commit message: PCBすすめた
Parts:
- RV1, RV2, RV3: footprint samacsys:SL4515NB103L15CM -> MyLibrary:SL4515G
- RV4: moved to B.Cu
- moved Q3 193.5 mm to (212.0, 79.5), turned to 90 degrees
- moved Q4 193.1 mm to (212.0, 86.6), turned to 90 degrees
- moved Q7 191.4 mm to (218.7, 76.5), turned to 90 degrees
- moved Q5 190.6 mm to (211.5, 100.3), turned to 90 degrees
- moved Q8 189.5 mm to (218.7, 89.6), turned to 90 degrees
- moved Q9 188.6 mm to (218.2, 97.3), turned to 90 degrees
- moved Q10 187.0 mm to (218.2, 110.4), turned to 90 degrees
- moved R34 184.0 mm to (224.2, 102.8), turned to 180 degrees
- moved R35 183.9 mm to (279.1, 150.0)
- moved R32 179.7 mm to (217.0, 82.0)
- moved R31 179.4 mm to (217.0, 79.0)
- moved U2 178.4 mm to (209.8, 59.8)
- moved RV4 177.6 mm to (224.6, 43.2)
- moved Q6 177.6 mm to (211.5, 107.4), turned to 90 degrees
- moved R33 176.3 mm to (216.5, 99.8)
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Other:
- board outline added: 100 x 70 mm

Commit message: 部品置いた
Parts:
- RV4: moved to F.Cu
- moved R35 118.1 mm to (187.6, 75.4), turned to -90 degrees
- moved R36 110.5 mm to (187.6, 90.7), turned to -90 degrees
- moved R25 95.1 mm to (164.1, 78.5)
- moved R21 94.5 mm to (164.1, 74.3)
- moved R26 88.6 mm to (164.1, 95.7)
- moved R22 83.7 mm to (164.1, 93.6)
- moved R23 82.9 mm to (164.1, 76.4)
- moved R24 78.3 mm to (164.1, 91.5)
- moved R19 75.7 mm to (181.8, 63.5), turned to -90 degrees
- moved Q9 41.6 mm to (177.8, 87.7), turned to 0 degrees
- moved Q7 41.1 mm to (177.8, 72.5), turned to 0 degrees
- moved R33 39.7 mm to (177.8, 91.1)
- moved R34 39.7 mm to (185.5, 94.1)
- moved Q5 39.7 mm to (172.8, 91.6)
- moved Q6 39.7 mm to (172.8, 98.7)
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Connections:
- C13 pad 2: Net-(U3C-+) -> Net-(U3D-+)
- J2 pad R: /outR -> /out_R
- J2 pad T: /outL -> /out_L
- R15 pad 2: Net-(U3C--) -> Net-(U3D--)
- R17 pad 1: Net-(U3C-+) -> Net-(U3D-+)
- R19 pad 1: Net-(U3D--) -> Net-(U3C--)
- R23 pad 2: /outR -> /out_L
- R24 pad 2: /outR -> /out_R
- R35 pad 2: /outR -> /out_L
- R36 pad 2: /outR -> /out_R
- R5 pad 2: Net-(U3D-+) -> Net-(U3C-+)
- RV1 pad 1: Net-(U3D--) -> Net-(U3C--)
- RV1 pad 3: Net-(U3D-+) -> Net-(U3C-+)
- RV2 pad 1: Net-(U3D--) -> Net-(U3C--)
- RV2 pad 3: Net-(U3D-+) -> Net-(U3C-+)
- RV3 pad 1: Net-(U3D--) -> Net-(U3C--)
- RV3 pad 3: Net-(U3D-+) -> Net-(U3C-+)
- U2 pad 3: /sigIN_R -> /sigIN_L
- U2 pad 5: /sigIN_L -> /sigIN_R
- U3 pad 14: Net-(R19-Pad2) -> Net-(U3D--)
- U3 pad 8: Net-(U3C--) -> Net-(R19-Pad2)

Commit message: gbr出力
Parts:
- added C15: 0.1u, Capacitor_THT:C_Disc_D5.1mm_W3.2mm_P5.00mm, F.Cu at (197.1, 78.1)
- added C16: 0.1u, Capacitor_THT:C_Disc_D5.1mm_W3.2mm_P5.00mm, F.Cu at (175.4, 62.0)
- added C17: 0.1u, Capacitor_THT:C_Disc_D5.1mm_W3.2mm_P5.00mm, F.Cu at (161.2, 78.5)
- added C18: 0.1u, Capacitor_THT:C_Disc_D5.1mm_W3.2mm_P5.00mm, F.Cu at (175.5, 107.9)
- added C19: 0.1u, Capacitor_THT:C_Disc_D5.1mm_W3.2mm_P5.00mm, F.Cu at (110.2, 92.6)
- added REF**: MountingHole_3.2mm_M3, MountingHole:MountingHole_3.2mm_M3, F.Cu at (196.6, 116.5)
- added REF**: MountingHole_3.2mm_M3, MountingHole:MountingHole_3.2mm_M3, F.Cu at (103.5, 116.5)
- added REF**: MountingHole_3.2mm_M3, MountingHole:MountingHole_3.2mm_M3, F.Cu at (103.5, 53.5)
- added SW1: SW_SPDT, samacsys:SS12D00G3, F.Cu at (101.5, 96.0)
- BT1: moved to B.Cu
- D1: footprint LED_THT:LED_D5.0mm -> LED_THT:LED_D3.0mm_Horizontal_O1.27mm_Z2.0mm
- moved R5 262.6 mm to (197.1, 75.1), turned to 180 degrees
- moved R6 253.8 mm to (197.1, 92.5), turned to 180 degrees
- moved D1 182.3 mm to (195.2, 112.3), turned to 90 degrees
- moved R1 164.4 mm to (191.0, 116.0), turned to 90 degrees
- moved BT1 66.5 mm to (115.0, 116.9), turned to 0 degrees
- moved R2 12.1 mm to (101.2, 91.0), turned to 90 degrees
- moved U2 5.40 mm to (190.8, 81.6)
- moved RV4 5.39 mm to (200.0, 56.0)
- moved C1 4.35 mm to (111.0, 67.0), turned to 90 degrees
- moved C2 3.38 mm to (111.0, 103.0), turned to 90 degrees
- moved R3 1.90 mm to (101.2, 84.0), turned to 90 degrees
- moved J1 0.40 mm to (197.9, 68.0)
Connections:
- BT1 pad 1: /V_{+} -> Net-(BT1-+)
- RV4 pad 1: Net-(R19-Pad2) -> Net-(R20-Pad2)
- RV4 pad 2: Net-(U4A-+) -> Net-(U4B-+)
- RV4 pad 4: Net-(R20-Pad2) -> Net-(R19-Pad2)
- RV4 pad 5: Net-(U4B-+) -> Net-(U4A-+)
- U5 pad 11: /V_{+} -> /V_{-}
Routing:
- net /V_{-}: track 0.00 -> 287.9 mm
- net /V_{+}: track 0.00 -> 272.8 mm
- net Net-(U3C-+): track 0.00 -> 122.9 mm, vias 0 -> 2
- net Net-(U5D--): track 0.00 -> 97.5 mm, vias 0 -> 1
- net Net-(U5D-+): track 0.00 -> 81.6 mm
- net Net-(U3C--): track 0.00 -> 60.1 mm
- net Net-(U4B-+): track 0.00 -> 52.6 mm, vias 0 -> 3
- net Net-(R20-Pad2): track 0.00 -> 51.7 mm, vias 0 -> 1
- net Net-(U4A-+): track 0.00 -> 49.6 mm, vias 0 -> 1
- net /out_L: track 0.00 -> 47.4 mm, vias 0 -> 1
- net Net-(C12-Pad1): track 0.00 -> 39.6 mm, vias 0 -> 1
- net Net-(C4-Pad1): track 0.00 -> 38.9 mm
- net Net-(C3-Pad1): track 0.00 -> 37.9 mm
- net /out_R: track 0.00 -> 36.0 mm
- net Net-(C11-Pad1): track 0.00 -> 35.8 mm, vias 0 -> 2
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- added copper zone on B.Cu, net GNDREF
- added copper zone on F.Cu, net GNDREF
Other:
- board text added: "100Hz"
- board text added: "10kHz"
- board text added: "1kHz"
- board text added: "AUDIO IN"
- board text added: "AUDIO OUT"
- board text added: "ON"
- board text added: "POWER"
- board text added: "VOLUME"

Commit message: シルク追記，gbr更新
Parts:
- added G***: LOGO, LOGO, B.Cu at (140.0, 85.0)
Other:
- board text added: "DESIGNED BY @Yu_san_T_robo"
- board text added: "EQUALIZER AMPLIFIRE v1.0"
