File: Earphones_amp.kicad_pcb (KiCad board)
At the start: 2 copper layers, 100 x 70 mm, 85 parts, among them J1 AudioJack3, J2 AudioJack3, Q1 2SC1815, Q10 PNP, Q2 2SA1015, Q3 PNP, Q4 NPN, Q5 PNP, Q6 NPN, Q7 NPN, Q8 PNP, Q9 NPN, SW1 SW_SPDT, U1 Opamp_Dual, U2 TL072, U3 TL074, U4 OPA1655DR, U5 TL074

Commit message: 回路図修正，v2.0に更新
Parts:
- removed REF** (x3): MountingHole_3.2mm_M3, MountingHole:MountingHole_3.2mm_M3
- added C20: 0.1u, Capacitor_THT:C_Disc_D4.7mm_W2.5mm_P5.00mm, F.Cu at (118.3, 74.1)
- added C21: 0.1u, Capacitor_THT:C_Disc_D4.7mm_W2.5mm_P5.00mm, F.Cu at (118.3, 100.9)
- added H1: MountingHole_Pad, MountingHole:MountingHole_3.2mm_M3_Pad_Via, F.Cu at (103.5, 53.5)
- added H2: MountingHole_Pad, MountingHole:MountingHole_3.2mm_M3_Pad_Via, F.Cu at (103.5, 116.5)
- added H3: MountingHole_Pad, MountingHole:MountingHole_3.2mm_M3_Pad_Via, F.Cu at (196.6, 116.5)
- added R37: 100k, Resistor_THT:R_Axial_DIN0204_L3.6mm_D1.6mm_P5.08mm_Horizontal, F.Cu at (192.1, 75.1)
- added R38: 100k, Resistor_THT:R_Axial_DIN0204_L3.6mm_D1.6mm_P5.08mm_Horizontal, F.Cu at (192.1, 77.2)
- D1: footprint LED_THT:LED_D3.0mm_Horizontal_O1.27mm_Z2.0mm -> LED_THT:LED_D5.0mm_Horizontal_O1.27mm_Z3.0mm
- R1: value 2k -> 10k
- moved D1 99.1 mm to (114.3, 55.0), turned to 180 degrees
- moved R1 95.5 mm to (115.5, 57.5), turned to 180 degrees
- moved SW1 20.8 mm to (110.0, 115.0)
- moved C15 4.24 mm to (197.1, 82.3)
- moved R5 4.24 mm to (197.1, 79.3)
- moved U2 4.20 mm to (190.8, 85.8)
- moved R6 3.58 mm to (197.1, 96.1)
- moved C1 2.50 mm to (108.5, 67.0)
- moved C2 2.50 mm to (108.5, 103.0)
Connections:
- Q10 pad 1: /V_{-} -> Net-(Q10-E)
- Q10 pad 2: Net-(Q10-C) -> /V_{-}
- Q3 pad 1: /V_{-} -> Net-(Q3-E)
- Q3 pad 2: Net-(Q3-C) -> /V_{-}
- Q5 pad 1: /V_{-} -> Net-(Q5-E)
- Q5 pad 2: Net-(Q5-C) -> /V_{-}
- Q7 pad 3: Net-(Q3-C) -> Net-(Q3-E)
- Q8 pad 1: /V_{-} -> Net-(Q8-E)
- Q8 pad 2: Net-(Q8-C) -> /V_{-}
- Q9 pad 3: Net-(Q5-C) -> Net-(Q5-E)
- R27 pad 2: Net-(Q3-C) -> Net-(Q3-E)
- R29 pad 2: Net-(Q5-C) -> Net-(Q5-E)
- R32 pad 2: Net-(Q8-C) -> Net-(Q8-E)
- R34 pad 2: Net-(Q10-C) -> Net-(Q10-E)
Routing:
- net /V_{-}: track 287.9 -> 313.5 mm
- net /V_{+}: track 272.8 -> 298.1 mm
- net Net-(BT1-+): track 26.5 -> 5.79 mm
- net Net-(Q5-C): track 13.9 -> 0.00 mm
- net Net-(Q3-C): track 12.8 -> 0.00 mm
- net Net-(Q3-E): track 0.00 -> 12.2 mm
- net /sigIN_R: track 21.4 -> 33.3 mm
- net Net-(Q5-E): track 0.00 -> 11.7 mm
- net /sigIN_L: track 24.8 -> 35.6 mm
- net Net-(Q8-C): track 9.36 -> 0.00 mm
- net Net-(Q10-E): track 0.00 -> 6.43 mm
- net Net-(Q8-E): track 0.00 -> 4.42 mm
- net Net-(Q10-C): track 4.39 -> 0.00 mm
- net Net-(U5D-+): track 81.6 -> 78.0 mm
- net Net-(D1-K): track 5.71 -> 3.03 mm
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Other:
- board text added: "EQUALIZER AMPLIFIRE v2.0"
- board text removed: "EQUALIZER AMPLIFIRE v1.0"
